File: Hardware/rover_car/rover_car.kicad_pcb (KiCad board)
At the start: 2 copper layers, 26 parts, among them J1 Conn_01x08_Female, J2 Conn_01x08_Female, M1 Motor_DC, M2 Motor_DC, M3 Motor_DC, M4 Motor_DC, M5 Motor_DC, M6 Motor_DC, U1 DRV8833PWP, U2 DRV8833PWP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

Commit message: PCB rover v0.1
Parts:
- removed J2: Conn_01x08_Female, Connector_PinHeader_2.54mm:PinHeader_1x08_P2.54mm_Vertical
- added J3: Screw_Terminal_01x02, TerminalBlock:TerminalBlock_bornier-2_P5.08mm, F.Cu at (144.0, 32.0)
- added R7: 200mOhms, Resistor_SMD:R_0805_2012Metric_Pad1.15x1.40mm_HandSolder, F.Cu at (156.9, 91.8)
- added R8: 200mOhm, Resistor_SMD:R_0805_2012Metric_Pad1.15x1.40mm_HandSolder, F.Cu at (156.1, 70.3)
- added R9: 200mOhms, Resistor_SMD:R_0805_2012Metric_Pad1.15x1.40mm_HandSolder, F.Cu at (157.0, 46.9)
- J1: value Conn_01x08_Female -> Conn_01x06_Female; footprint Connector_PinHeader_2.54mm:PinHeader_1x08_P2.54mm_Vertical -> Connector_PinSocket_2.54mm:PinSocket_1x06_P2.54mm_Vertical
- M1, M2, M3, M4, M5, M6: footprint TerminalBlock:TerminalBlock_Altech_AK300-2_P5.00mm -> TerminalBlock:TerminalBlock_bornier-2_P5.08mm
- moved M1 79.9 mm to (164.8, 87.9), turned to 270 degrees
- moved M2 65.3 mm to (164.9, 77.3)
- moved M3 61.6 mm to (164.9, 66.6), turned to 270 degrees
- moved R1 61.3 mm to (156.9, 89.9), turned to 180 degrees
- moved C1 59.9 mm to (143.7, 85.0), turned to 270 degrees
- moved U1 59.4 mm to (154.4, 85.4)
- moved M5 56.4 mm to (164.9, 45.6), turned to 270 degrees
- moved R3 55.6 mm to (156.5, 79.5), turned to 270 degrees
- moved C3 54.5 mm to (148.1, 87.2), turned to 90 degrees
- moved C2 54.4 mm to (145.8, 85.0)
- moved M4 43.8 mm to (164.9, 56.1)
- moved M6 40.1 mm to (164.9, 35.0)
- moved J1 22.5 mm to (137.0, 61.4)
- moved C6 18.1 mm to (147.6, 65.0), turned to 90 degrees
- moved R4 17.6 mm to (156.0, 58.5), turned to 270 degrees
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Connections:
- J1 pad 1: /GPIO4 -> GND
- J1 pad 2: /GPIO2 -> /GPIO14
- J1 pad 3: /GPIO14 -> /GPIO15
- J1 pad 4: /GPIO15 -> /GPIO4
- J1 pad 5: /GPIO13 -> /GPIO2
- J1 pad 6: /GPIO12 -> VCC
- M1 pad 1: /AOUT1 -> /AOUT2
- M1 pad 2: /AOUT2 -> /AOUT1
- M3 pad 1: /AFDER1 -> /AFDER2
- M3 pad 2: /AFDER2 -> /AFDER1
- M5 pad 1: /ADER1 -> /ADER2
- M5 pad 2: /ADER2 -> /ADER1
- R3 pad 1: +5V -> VCC
- R4 pad 1: +5V -> VCC
- R6 pad 1: +5V -> VCC
- U1 pad 3: Net-(R1-Pad1) -> Net-(R7-Pad1)
- U2 pad 10: /GPIO3 -> /GPIO15
- U2 pad 15: /GPIO13 -> /GPIO2
- U2 pad 16: /GPIO12 -> /GPIO4
- U2 pad 3: Net-(R2-Pad1) -> Net-(R8-Pad1)
- U2 pad 9: /GPIO1 -> /GPIO14
- U3 pad 3: Net-(R5-Pad1) -> Net-(R9-Pad1)
Routing:
- net GND: track 0.00 -> 94.1 mm
- net +12V: track 0.00 -> 93.8 mm
- net VCC: track 0.00 -> 67.0 mm, vias 0 -> 4
- net /GPIO2: track 0.00 -> 53.5 mm, vias 0 -> 3
- net /GPIO4: track 0.00 -> 50.7 mm, vias 0 -> 3
- net /GPIO14: track 0.00 -> 50.3 mm, vias 0 -> 3
- net /GPIO15: track 0.00 -> 45.7 mm, vias 0 -> 3
- net Net-(C7-Pad2): track 0.00 -> 16.4 mm, vias 0 -> 2
- net Net-(C4-Pad2): track 0.00 -> 15.1 mm, vias 0 -> 2
- net Net-(C1-Pad2): track 0.00 -> 14.6 mm, vias 0 -> 2
- net /BFDER1: track 0.00 -> 13.5 mm
- net /BOUT1: track 0.00 -> 13.3 mm
- net /BDER1: track 0.00 -> 12.8 mm
- net /ADER1: track 0.00 -> 12.1 mm
- net /AFDER1: track 0.00 -> 12.0 mm
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- added copper zone on B.Cu, net GND
- added copper zone on F.Cu, net GND
Other:
- board outline added: 36.8 x 71.1 mm
- net class Default: clearance 0.2 -> 0.25; trace_width 0.25 -> 0.3
- net class VCC+ added: clearance 0.5, trace_width 0.7, via_dia 0.8, via_drill 0.4
- net class vcc added: clearance 0.5, trace_width 0.7, via_dia 0.8, via_drill 0.4
- rule trace_clearance: 0.2 -> 0.25

Commit message: Add capacitor
Parts:
- C2, C8: footprint Capacitor_SMD:C_0805_2012Metric_Pad1.15x1.40mm_HandSolder -> Capacitor_SMD:CP_Elec_4x5.4
- C5: footprint Capacitor_SMD:C_0805_2012Metric_Pad1.15x1.40mm_HandSolder -> Capacitor_SMD:C_Elec_4x5.4
- moved C5 22.6 mm to (140.1, 84.7)
- moved C2 21.5 mm to (143.3, 63.6)
- moved C4 3.27 mm to (146.8, 63.0)
- moved C1 1.81 mm to (145.4, 84.3)
- moved C9 1.71 mm to (149.2, 45.0)
- moved C6 1.46 mm to (148.8, 65.9)
- moved C7 1.33 mm to (141.7, 43.3)
- moved C3 1.11 mm to (149.2, 87.0)
- moved C8 1.06 mm to (145.5, 42.3)
Routing:
- net GND: track 94.1 -> 105.0 mm
- net +12V: track 93.8 -> 104.4 mm
- net Net-(C4-Pad2): track 15.1 -> 11.9 mm
- net Net-(C9-Pad1): track 5.34 -> 3.88 mm
- net Net-(C1-Pad2): track 14.6 -> 13.1 mm
- net Net-(C3-Pad1): track 4.34 -> 3.49 mm
- net Net-(C6-Pad1): track 4.40 -> 3.81 mm
- net Net-(C7-Pad2): track 16.4 -> 17.0 mm

Commit message: Last Revision pcb
Parts:
- moved C7 5.81 mm to (147.2, 41.4), turned to 90 degrees
- moved C8 3.44 mm to (142.9, 44.5)
- moved C4 2.50 mm to (146.8, 60.5), turned to 90 degrees
- moved C5 2.39 mm to (142.4, 85.0)
- moved C1 2.29 mm to (147.4, 83.3), turned to 90 degrees
Routing:
- net Net-(C7-Pad2): track 17.0 -> 5.27 mm, vias 2 -> 0
- net +12V: track 104.4 -> 96.5 mm
- net Net-(C1-Pad2): track 13.1 -> 5.51 mm, vias 2 -> 0
- net Net-(C4-Pad2): track 11.9 -> 5.99 mm, vias 2 -> 0
- net GND: track 105.0 -> 104.1 mm

Commit message: Last revision
Parts:
- removed R3, R4, R6: 1KOhm, Resistor_SMD:R_0805_2012Metric_Pad1.15x1.40mm_HandSolder
- moved R9 0.76 mm to (157.1, 47.7)
- moved R5 0.60 mm to (157.1, 49.6)
- moved R7 0.43 mm to (156.9, 92.2)
- moved R1 0.40 mm to (156.9, 90.3)
Connections:
- U1 pad 1: GND -> VCC
- U2 pad 1: GND -> VCC
- U3 pad 1: GND -> VCC
Routing:
- net GND: track 104.1 -> 94.6 mm
- net Net-(R7-Pad1): track 8.06 -> 11.5 mm
- net Net-(U2-Pad8): track 3.20 -> 0.00 mm
- net VCC: track 67.0 -> 70.2 mm, vias 4 -> 3
- net Net-(U1-Pad8): track 2.95 -> 0.00 mm
- net Net-(R1-Pad1): track 7.40 -> 10.2 mm
- net Net-(U3-Pad8): track 2.70 -> 0.00 mm
- net Net-(R5-Pad1): track 10.2 -> 12.9 mm
- net Net-(R9-Pad1): track 4.68 -> 6.63 mm
- net Net-(R2-Pad1): track 7.78 -> 8.52 mm

Commit message: Accommodation revision
Parts:
- added REF**: MountingHole_3.2mm_M3_Pad_Via, MountingHole:MountingHole_3.2mm_M3_Pad_Via, F.Cu at (157.3, 34.7)
- added REF**: MountingHole_3.2mm_M3_Pad_Via, MountingHole:MountingHole_3.2mm_M3_Pad_Via, F.Cu at (139.3, 92.8)
- added REF**: MountingHole_3.2mm_M3_Pad_Via, MountingHole:MountingHole_3.2mm_M3_Pad_Via, F.Cu at (139.4, 34.8)
- moved J3 1.92 mm to (145.9, 32.3)
- moved C5 1.48 mm to (143.9, 84.7)
- moved C4 1.23 mm to (147.4, 61.5)
- moved C8 1.10 mm to (143.9, 44.1)
- moved R2 0.85 mm to (156.9, 68.4)
- moved R8 0.85 mm to (156.9, 70.3)
- moved C2 0.55 mm to (143.9, 63.6)
- moved C7 0.32 mm to (147.4, 41.2)
- moved U2 0.22 mm to (154.4, 63.7)
- moved U3 0.16 mm to (154.4, 42.8)
- moved R5 0.12 mm to (156.9, 49.6)
- moved R9 0.12 mm to (156.9, 47.7)
Routing:
- net GND: track 94.6 -> 89.2 mm
- net +12V: track 96.5 -> 92.7 mm
- net /GPIO14: track 50.3 -> 49.5 mm
- net Net-(R8-Pad1): track 10.4 -> 9.76 mm
Other:
- board text added: "5V"
- board text added: "GND"
- board text added: "PWM1"
- board text added: "PWM2"
- board text added: "PWM3"
- board text added: "PWM4"

Commit message: Last revision pcb
Parts:
- added REF**: MountingHole_3.2mm_M3_Pad_Via, MountingHole:MountingHole_3.2mm_M3_Pad_Via, F.Cu at (156.0, 93.0)
- moved J3 19.4 mm to (137.4, 49.8), turned to 270 degrees
- moved R7 12.8 mm to (156.9, 79.4)
- moved R8 12.7 mm to (156.9, 57.6)
- moved R1 8.90 mm to (156.9, 81.4)
- moved R2 8.80 mm to (156.9, 59.6)
- moved M1 3.00 mm to (167.8, 87.9)
- moved M2 3.00 mm to (167.9, 77.3)
- moved M3 3.00 mm to (167.9, 66.6)
- moved M4 3.00 mm to (167.9, 56.1)
- moved M5 3.00 mm to (167.9, 45.6)
- moved M6 3.00 mm to (167.9, 35.0)
- moved REF** 1.33 mm to (156.0, 35.0)
- moved REF** 0.46 mm to (139.0, 35.0)
- moved REF** 0.40 mm to (139.0, 93.0)
Connections:
- net /GPIO2 renamed /GPIO12
Routing:
- net GND: track 89.2 -> 109.6 mm
- net +12V: track 92.7 -> 86.2 mm
- net Net-(R1-Pad1): track 10.2 -> 5.63 mm
- net Net-(R8-Pad1): track 9.76 -> 13.0 mm
- net /BOUT2: track 8.83 -> 11.8 mm
- net /BOUT1: track 13.3 -> 16.3 mm
- net /BFDER2: track 9.09 -> 12.1 mm
- net /BFDER1: track 13.5 -> 16.5 mm
- net /AOUT2: track 8.56 -> 11.6 mm
- net /AOUT1: track 10.5 -> 13.5 mm
- net /AFDER2: track 9.89 -> 12.9 mm
- net /AFDER1: track 12.0 -> 15.0 mm
- net /ADER2: track 8.61 -> 11.6 mm
- net /ADER1: track 12.1 -> 15.1 mm
- net /BDER2: track 8.87 -> 11.9 mm
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Other:
- board size 36.8 x 71.1 mm -> 40 x 70 mm
- board text added: "+"
- board text added: "-"

Commit message: Track revision
Parts:
- moved R5 6.63 mm to (155.6, 43.1)
- moved R9 6.63 mm to (155.6, 41.2)
- moved C9 5.81 mm to (147.8, 50.6)
- moved C7 5.14 mm to (147.0, 46.3)
- moved C8 5.00 mm to (144.1, 49.1)
- moved J3 4.37 mm to (137.1, 45.4)
- moved U3 4.37 mm to (153.7, 47.1)
- moved U1 0.62 mm to (153.8, 85.4)
- moved U2 0.62 mm to (153.8, 63.7)
Routing:
- net GND: track 109.6 -> 53.6 mm
- net /GPIO14: track 49.6 -> 39.3 mm
- net Net-(R5-Pad1): track 12.9 -> 6.52 mm
- net +12V: track 86.2 -> 80.5 mm
- net Net-(R9-Pad1): track 6.63 -> 11.9 mm
- net /BDER1: track 14.5 -> 18.4 mm
- net VCC: track 70.2 -> 66.5 mm
- net /GPIO4: track 49.2 -> 46.0 mm
- net /ADER1: track 15.1 -> 12.3 mm
- net /BDER2: track 11.9 -> 14.4 mm
- net Net-(C9-Pad1): track 3.88 -> 6.05 mm
- net Net-(C4-Pad2): track 5.60 -> 4.29 mm
- net Net-(C7-Pad2): track 5.52 -> 4.24 mm
- net /ADER2: track 11.6 -> 12.6 mm
- net Net-(R1-Pad1): track 5.63 -> 6.51 mm
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
Commit message: Change tracks
Parts:
- moved R5 1.33 mm to (156.9, 43.1)
- moved R9 1.33 mm to (156.9, 41.2)
- moved C8 0.15 mm to (143.9, 49.1)
- moved U3 0.10 mm to (153.8, 47.1)
Routing:
- net +12V: track 80.5 -> 99.3 mm
Other:
- net class VCC+: trace_width 0.7 -> 1.2
Changed lines of the file:
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@@
-(kicad_pcb (version 20171130) (host pcbnew "(5.1.2)-2")
+(kicad_pcb (version 20171130) (host pcbnew "(5.1.2)-1")
   (general
     (thickness 1.6)
     (drawings 22)
-    (tracks 416)
+    (tracks 420)
     (zones 0)
     (modules 30)
@@
   (net_class VCC+ ""
     (clearance 0.5)
-    (trace_width 0.7)
+    (trace_width 1.2)
     (via_dia 0.8)
     (via_drill 0.4)
     (uvia_dia 0.3)
     (uvia_drill 0.1)
+    (add_net +12V)
   )
   (net_class vcc ""
@@
     (uvia_dia 0.3)
     (uvia_drill 0.1)
-    (add_net +12V)
   )
   (module TerminalBlock:TerminalBlock_bornier-2_P5.08mm (layer F.Cu)
@@
   )
   (module Package_SO:HTSSOP-16-1EP_4.4x5mm_P0.65mm_EP3.4x5mm_Mask2.46x2.31mm_ThermalVias (layer F.Cu)
-    (at 153.675 47.1 180)
+    (at 153.775 47.1 180)
     (descr "16-Lead Plastic HTSSOP (4.4x5x1.2mm); Thermal pad with vias; (http://www.ti.com/lit/ds/symlink/drv8833.pdf)")
     (tags "SSOP 0.65")
@@
   )
   (module Resistor_SMD:R_0805_2012Metric_Pad1.15x1.40mm_HandSolder (layer F.Cu)
-    (at 155.6 43.1 180)
+    (at 156.925 43.1 180)
     (descr "Resistor SMD 0805 (2012 Metric), square (rectangular) end terminal, IPC_7351 nominal with elongated pad for handsoldering. (Body size source: https://docs.google.com/spreadsheets/d/1BsfQQcO9C6DZCsRaXUlFlo91Tg2WpOkGARC1WS5S8t0/edit?usp=sharing), generated with kicad-footprint-generator")
     (tags "resistor handsolder")
@@
   )
   (module Resistor_SMD:R_0805_2012Metric_Pad1.15x1.40mm_HandSolder (layer F.Cu)
-    (at 155.6 41.2 180)
+    (at 156.925 41.2 180)
     (descr "Resistor SMD 0805 (2012 Metric), square (rectangular) end terminal, IPC_7351 nominal with elongated pad for handsoldering. (Body size source: https://docs.google.com/spreadsheets/d/1BsfQQcO9C6DZCsRaXUlFlo91Tg2WpOkGARC1WS5S8t0/edit?usp=sharing), generated with kicad-footprint-generator")
     (tags "resistor handsolder")
@@
   )
   (module Capacitor_SMD:CP_Elec_4x5.4 (layer F.Cu)
-    (at 144.05 49.15 270)
+    (at 143.9 49.15 270)
     (descr "SMD capacitor, aluminum electrolytic, Panasonic A5 / Nichicon, 4.0x5.4mm")
     (tags "capacitor electrolytic")
@@
   (segment (start 151.625 85.09) (end 150.365 85.09) (width 0.3) (layer F.Cu) (net 1))
   (segment (start 150.365 85.09) (end 149.9 84.625) (width 0.3) (layer F.Cu) (net 1))
-  (segment (start 144.7 83.05) (end 145.65 83.05) (width 0.7) (layer F.Cu) (net 1))
   (segment (start 139.9 61.722) (end 139.9 60.9) (width 0.7) (layer F.Cu) (net 1))
   (segment (start 139.9 61.722) (end 140.328 61.722) (width 0.7) (layer F.Cu) (net 1))
@@
   (segment (start 149.614357 63.296416) (end 148.446416 63.296416) (width 0.7) (layer F.Cu) (net 1))
   (segment (start 148.446416 63.296416) (end 147.575 62.425) (width 0.7) (layer F.Cu) (net 1))
-  (segment (start 143.6 83.05) (end 145.175 83.05) (width 0.7) (layer F.Cu) (net 1))
   (segment (start 144.05 47.35) (end 143.15 47.35) (width 0.7) (layer F.Cu) (net 1))
-  (segment (start 140.9 49.475) (end 141.025 49.475) (width 0.3) (layer F.Cu) (net 1))
-  (segment (start 144.05 47.35) (end 147 47.35) (width 0.7) (layer F.Cu) (net 1))
   (segment (start 147 47.35) (end 148.475 47.35) (width 0.7) (layer F.Cu) (net 1))
   (segment (start 148.475 47.35) (end 149.05 46.775) (width 0.7) (layer F.Cu) (net 1))
@@
   (segment (start 150.9 46.775) (end 150.075 46.775) (width 0.3) (layer F.Cu) (net 1))
   (segment (start 147.225 84.625) (end 149.55 84.625) (width 0.7) (layer F.Cu) (net 1))
-  (segment (start 145.78 83.18) (end 147.225 84.625) (width 0.7) (layer F.Cu) (net 1))
-  (segment (start 145.78 75.055) (end 145.78 83.18) (width 0.7) (layer F.Cu) (net 1))
-  (segment (start 139.95 69.225) (end 145.78 75.055) (width 0.7) (layer F.Cu) (net 1))
   (segment (start 139.9 62.4) (end 139.95 62.45) (width 0.7) (layer F.Cu) (net 1))
   (segment (start 139.95 62.45) (end 139.95 69.225) (width 0.7) (layer F.Cu) (net 1))
-  (segment (start 139.9 60.9) (end 141.025 59.775) (width 0.7) (layer F.Cu) (net 1))
-  (segment (start 141.025 59.775) (end 141.025 50.075) (width 0.7) (layer F.Cu) (net 1))
-  (segment (start 141.025 50.075) (end 141.025 49.425) (width 0.7) (layer F.Cu) (net 1))
-  (segment (start 137.1 45.425) (end 139.3 45.425) (width 0.7) (layer F.Cu) (net 1))
-  (segment (start 139.3 45.425) (end 141.025 47.15) (width 0.7) (layer F.Cu) (net 1))
-  (segment (start 141.025 48.3) (end 141.025 48.15) (width 0.7) (layer F.Cu) (net 1))
-  (segment (start 141.025 48.3) (end 141.025 50.075) (width 0.7) (layer F.Cu) (net 1))
   (segment (start 143.1 47.35) (end 144.05 47.35) (width 0.7) (layer F.Cu) (net 1))
   (segment (start 142.225 47.35) (end 143.1 47.35) (width 0.7) (layer F.Cu) (net 1))
-  (segment (start 141.375 47.35) (end 141.025 47.7) (width 0.7) (layer F.Cu) (net 1))
-  (segment (start 141.025 47.15) (end 141.025 47.7) (width 0.7) (layer F.Cu) (net 1))
-  (segment (start 141.025 47.7) (end 141.025 48.3) (width 0.7) (layer F.Cu) (net 1))
-  (segment (start 141.775 47.55) (end 141.025 48.3) (width 0.7) (layer F.Cu) (net 1))
-  (segment (start 141.775 47.35) (end 141.775 47.55) (width 0.7) (layer F.Cu) (net 1))
-  (segment (start 142.225 47.35) (end 141.775 47.35) (width 0.7) (layer F.Cu) (net 1))
-  (segment (start 141.775 47.35) (end 141.375 47.35) (width 0.7) (layer F.Cu) (net 1))
+  (segment (start 139.9 79.025) (end 143.9 83.025) (width 1.2) (layer F.Cu) (net 1))
+  (segment (start 139.9 69.175) (end 139.9 79.025) (width 1.2) (layer F.Cu) (net 1))
+  (segment (start 147 47.35) (end 144.05 47.35) (width 1.2) (layer F.Cu) (net 1))
+  (segment (start 142.975 61.875) (end 139.9 61.875) (width 1.2) (layer F.Cu) (net 1))
+  (segment (start 143 61.85) (end 142.975 61.875) (width 1.2) (layer F.Cu) (net 1))
+  (segment (start 143.9 61.85) (end 143 61.85) (width 1.2) (layer F.Cu) (net 1))
+  (segment (start 139.9 60.9) (end 139.9 61.875) (width 1.2) (layer F.Cu) (net 1))
+  (segment (start 139.9 61.875) (end 139.9 69.175) (width 1.2) (layer F.Cu) (net 1))
+  (segment (start 139.95 60.85) (end 139.9 60.9) (width 1.2) (layer F.Cu) (net 1))
+  (segment (start 139.95 50.125) (end 139.95 51.3) (width 1.2) (layer F.Cu) (net 1))
+  (segment (start 139.95 51.3) (end 139.95 60.85) (width 1.2) (layer F.Cu) (net 1))
+  (segment (start 137.1 45.425) (end 138.55 45.425) (width 1.2) (layer F.Cu) (net 1))
+  (segment (start 138.55 45.425) (end 139.95 46.825) (width 1.2) (layer F.Cu) (net 1))
+  (segment (start 138.55 45.425) (end 140.475 47.35) (width 1.2) (layer F.Cu) (net 1))
+  (segment (start 140.225 48.85) (end 141.725 47.35) (width 1.2) (layer F.Cu) (net 1))
+  (segment (start 139.95 48.85) (end 140.225 48.85) (width 1.2) (layer F.Cu) (net 1))
+  (segment (start 141.725 47.35) (end 144.05 47.35) (width 1.2) (layer F.Cu) (net 1))
+  (segment (start 140.475 47.35) (end 141.725 47.35) (width 1.2) (layer F.Cu) (net 1))
+  (segment (start 139.95 46.825) (end 139.95 48.85) (width 1.2) (layer F.Cu) (net 1))
+  (segment (start 139.95 48.85) (end 139.95 51.3) (width 1.2) (layer F.Cu) (net 1))
+  (segment (start 144.525 62.55) (end 147.375 62.55) (width 1.2) (layer F.Cu) (net 1))
+  (segment (start 146.625 84.3) (end 147.425 84.3) (width 1.2) (layer F.Cu) (net 1))
+  (segment (start 146.22071 83.89571) (end 146.625 84.3) (width 1.2) (layer F.Cu) (net 1))
+  (segment (start 144.77071 83.89571) (end 146.22071 83.89571) (width 1.2) (layer F.Cu) (net 1))
+  (segment (start 143.9 83.025) (end 144.77071 83.89571) (width 1.2) (layer F.Cu) (net 1))
   (segment (start 147.515685 82.425) (end 146.95 82.425) (width 0.3) (layer F.Cu) (net 2))
   (segment (start 151.625 84.44) (end 150.677165 84.44) (width 0.3) (layer F.Cu) (net 2))
