File: Hardware/rover_car/rover_car.sch (KiCad schematic (older format))
At the start: 26 parts, among them J1 Conn_01x08_Female, J2 Conn_01x08_Female, M1 Motor_DC, M2 Motor_DC, M3 Motor_DC, M4 Motor_DC, M5 Motor_DC, M6 Motor_DC, U1 DRV8833PWP, U2 DRV8833PWP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

Commit message: At schematic
Parts:
- C1, C4, C7: value C_Small -> .01uF
- C2, C5, C8: value CP1_Small -> 10uF
- C3, C6, C9: value C_Small -> 2.2uF
- R1: value R_Small -> 20mOhms
- R2, R5: value R_Small -> 200mOhm
- R3, R4, R6: value R_Small -> 1KOhm
Changed lines of the file:
@@
 P 1850 1350
 F 0 "C1" H 1942 1396 50  0000 L CNN
-F 1 "C_Small" H 1942 1305 50  0000 L CNN
+F 1 ".01uF" H 1942 1305 50  0000 L CNN
 F 2 "" H 1850 1350 50  0001 C CNN
 F 3 "~" H 1850 1350 50  0001 C CNN
@@
 P 2150 1200
 F 0 "C2" H 2241 1246 50  0000 L CNN
-F 1 "CP1_Small" H 2241 1155 50  0000 L CNN
+F 1 "10uF" H 2241 1155 50  0000 L CNN
 F 2 "" H 2150 1200 50  0001 C CNN
 F 3 "~" H 2150 1200 50  0001 C CNN
@@
 P 3350 1350
 F 0 "C3" H 3442 1396 50  0000 L CNN
-F 1 "C_Small" H 3442 1305 50  0000 L CNN
+F 1 "2.2uF" H 3442 1305 50  0000 L CNN
 F 2 "" H 3350 1350 50  0001 C CNN
 F 3 "~" H 3350 1350 50  0001 C CNN
@@
 U 1 1 5D1E7C75
 P 1650 2100
-F 0 "R1" H 1709 2146 50  0000 L CNN
-F 1 "R_Small" H 1709 2055 50  0000 L CNN
+F 0 "R1" V 1450 2100 50  0000 L CNN
+F 1 "20mOhms" V 1550 1950 50  0000 L CNN
 F 2 "" H 1650 2100 50  0001 C CNN
 F 3 "~" H 1650 2100 50  0001 C CNN
@@
 P 6500 1450
 F 0 "C7" H 6592 1496 50  0000 L CNN
-F 1 "C_Small" H 6592 1405 50  0000 L CNN
+F 1 ".01uF" H 6592 1405 50  0000 L CNN
 F 2 "" H 6500 1450 50  0001 C CNN
 F 3 "~" H 6500 1450 50  0001 C CNN
@@
 P 6800 1300
 F 0 "C8" H 6891 1346 50  0000 L CNN
-F 1 "CP1_Small" H 6891 1255 50  0000 L CNN
+F 1 "10uF" H 6891 1255 50  0000 L CNN
 F 2 "" H 6800 1300 50  0001 C CNN
 F 3 "~" H 6800 1300 50  0001 C CNN
@@
 P 8000 1450
 F 0 "C9" H 8092 1496 50  0000 L CNN
-F 1 "C_Small" H 8092 1405 50  0000 L CNN
+F 1 "2.2uF" H 8092 1405 50  0000 L CNN
 F 2 "" H 8000 1450 50  0001 C CNN
 F 3 "~" H 8000 1450 50  0001 C CNN
@@
 U 1 1 5D1F7E9A
 P 6300 2200
-F 0 "R5" H 6359 2246 50  0000 L CNN
-F 1 "R_Small" H 6359 2155 50  0000 L CNN
+F 0 "R5" V 6100 2150 50  0000 L CNN
+F 1 "200mOhm" V 6200 2000 50  0000 L CNN
 F 2 "" H 6300 2200 50  0001 C CNN
 F 3 "~" H 6300 2200 50  0001 C CNN
@@
 P 3600 4750
 F 0 "C4" H 3692 4796 50  0000 L CNN
-F 1 "C_Small" H 3692 4705 50  0000 L CNN
+F 1 ".01uF" H 3692 4705 50  0000 L CNN
 F 2 "" H 3600 4750 50  0001 C CNN
 F 3 "~" H 3600 4750 50  0001 C CNN
@@
 P 3900 4600
 F 0 "C5" H 3991 4646 50  0000 L CNN
-F 1 "CP1_Small" H 3991 4555 50  0000 L CNN
+F 1 "10uF" H 3991 4555 50  0000 L CNN
 F 2 "" H 3900 4600 50  0001 C CNN
 F 3 "~" H 3900 4600 50  0001 C CNN
@@
 P 5100 4750
 F 0 "C6" H 5192 4796 50  0000 L CNN
-F 1 "C_Small" H 5192 4705 50  0000 L CNN
+F 1 "2.2uF" H 5192 4705 50  0000 L CNN
 F 2 "" H 5100 4750 50  0001 C CNN
 F 3 "~" H 5100 4750 50  0001 C CNN
@@
 U 1 1 5D2161EF
 P 3400 5500
-F 0 "R2" H 3459 5546 50  0000 L CNN
-F 1 "R_Small" H 3459 5455 50  0000 L CNN
+F 0 "R2" V 3250 5450 50  0000 L CNN
+F 1 "200mOhm" V 3300 5350 50  0000 L CNN
 F 2 "" H 3400 5500 50  0001 C CNN
 F 3 "~" H 3400 5500 50  0001 C CNN
@@
 P 3550 1800
 F 0 "R3" H 3609 1846 50  0000 L CNN
-F 1 "R_Small" H 3609 1755 50  0000 L CNN
+F 1 "1KOhm" H 3609 1755 50  0000 L CNN
 F 2 "" H 3550 1800 50  0001 C CNN
 F 3 "~" H 3550 1800 50  0001 C CNN
@@
 P 8200 1900
 F 0 "R6" H 8259 1946 50  0000 L CNN
-F 1 "R_Small" H 8259 1855 50  0000 L CNN
+F 1 "1KOhm" H 8259 1855 50  0000 L CNN
 F 2 "" H 8200 1900 50  0001 C CNN
 F 3 "~" H 8200 1900 50  0001 C CNN
@@
 P 5300 5200
 F 0 "R4" H 5359 5246 50  0000 L CNN
-F 1 "R_Small" H 5359 5155 50  0000 L CNN
+F 1 "1KOhm" H 5359 5155 50  0000 L CNN
 F 2 "" H 5300 5200 50  0001 C CNN
 F 3 "~" H 5300 5200 50  0001 C CNN

Commit message: Add pcb and edit sch
Parts:
- C1, C4, C7: footprint (none) -> Capacitor_SMD:C_0805_2012Metric_Pad1.15x1.40mm_HandSolder; manf# (none) -> 710-885012207039
- C2, C5, C8: footprint (none) -> Capacitor_SMD:C_0805_2012Metric_Pad1.15x1.40mm_HandSolder; manf# (none) -> 755-TCTP1C106M8R
- C3, C6, C9: footprint (none) -> Capacitor_SMD:C_0805_2012Metric_Pad1.15x1.40mm_HandSolder; manf# (none) -> 710-885012107012
- J1, J2: footprint (none) -> Connector_PinHeader_2.54mm:PinHeader_1x08_P2.54mm_Vertical
- M1, M2, M3, M4, M5, M6: footprint (none) -> TerminalBlock:TerminalBlock_Altech_AK300-2_P5.00mm
- R1: value 20mOhms -> 200mOhms; footprint (none) -> Resistor_SMD:R_0805_2012Metric_Pad1.15x1.40mm_HandSolder; manf# (none) -> 667-ERJ-U6SFR20V
- R2, R5: footprint (none) -> Resistor_SMD:R_0805_2012Metric_Pad1.15x1.40mm_HandSolder; manf# (none) -> 667-ERJ-U6SFR20V
- R3, R4, R6: footprint (none) -> Resistor_SMD:R_0805_2012Metric_Pad1.15x1.40mm_HandSolder; manf# (none) -> 660-RN73H2ATD1001B25
- U1, U2, U3: manf# (none) -> 595-DRV8833CPWPR

Commit message: PCB rover v0.1
Parts:
- removed J1, J2: Conn_01x08_Female, Connector_PinHeader_2.54mm:PinHeader_1x08_P2.54mm_Vertical, symbol Connector:Conn_01x08_Female
- added J1: Conn_01x06_Female, Connector_PinSocket_2.54mm:PinSocket_1x06_P2.54mm_Vertical, symbol Connector:Conn_01x06_Female
- added J3: Screw_Terminal_01x02, TerminalBlock:TerminalBlock_bornier-2_P5.08mm, symbol Connector:Screw_Terminal_01x02
- added R7, R9: 200mOhms, Resistor_SMD:R_0805_2012Metric_Pad1.15x1.40mm_HandSolder, symbol Device:R_Small
- added R8: 200mOhm, Resistor_SMD:R_0805_2012Metric_Pad1.15x1.40mm_HandSolder, symbol Device:R_Small
- M1, M2, M3, M4, M5, M6: footprint TerminalBlock:TerminalBlock_Altech_AK300-2_P5.00mm -> TerminalBlock:TerminalBlock_bornier-2_P5.08mm
Connections:
- net GPIO1 is gone; now on net GPIO14: U2.9 (BIN1)
- net GPIO12 is gone; now on net GPIO4: U2.16 (AIN1)
- net GPIO13 is gone; now on net GPIO2: U2.15 (AIN2)
- net GPIO3 is gone; now on net GPIO15: U2.10 (BIN2)
- net +12V: now also J3.1 (Pin_1)
- net ADER1: now also M5.2 (-); no longer M5.1 (+)
- net ADER2: now also M5.1 (+); no longer M5.2 (-)
- net AFDER1: now also M3.2 (-); no longer M3.1 (+)
- net AFDER2: now also M3.1 (+); no longer M3.2 (-)
- net AOUT1: now also M1.2 (-); no longer M1.1 (+)
- net AOUT2: now also M1.1 (+); no longer M1.2 (-)
- net GND: now also J1.1 (Pin_1), J3.2 (Pin_2), R7.2, R8.2, R9.2
- net GPIO14: now also J1.2 (Pin_2)
- net GPIO15: now also J1.3 (Pin_3)
- net GPIO2: now also J1.5 (Pin_5)
- net GPIO4: now also J1.4 (Pin_4)
- net at R1.1, U1.6 (BISEN): no longer U1.3 (AISEN)
- net at R5.1, U3.6 (BISEN): no longer U3.3 (AISEN)
- net at R2.1, U2.6 (BISEN): no longer U2.3 (AISEN)
- net +5V renamed VCC
- net VCC: now also J1.6 (Pin_6)
- new net: R7.1, U1.3 (AISEN)
- new net: R9.1, U3.3 (AISEN)
- new net: R8.1, U2.3 (AISEN)
Other:
- note added: "ENTRADA DE VOLTAJE"

Commit message: Add capacitor
Parts:
- C2, C8: footprint Capacitor_SMD:C_0805_2012Metric_Pad1.15x1.40mm_HandSolder -> Capacitor_SMD:CP_Elec_4x5.4; manf# 755-TCTP1C106M8R -> 865090440003
- C5: footprint Capacitor_SMD:C_0805_2012Metric_Pad1.15x1.40mm_HandSolder -> Capacitor_SMD:C_Elec_4x5.4; manf# 755-TCTP1C106M8R -> 865090440003
Changed lines of the file:
@@
 F 0 "C2" H 2241 1246 50  0000 L CNN
 F 1 "10uF" H 2241 1155 50  0000 L CNN
-F 2 "Capacitor_SMD:C_0805_2012Metric_Pad1.15x1.40mm_HandSolder" H 2150 1200 50  0001 C CNN
-F 3 "https://www.mouser.mx/datasheet/2/348/tct_p-951873.pdf" H 2150 1200 50  0001 C CNN
-F 4 "755-TCTP1C106M8R" H 2150 1200 50  0001 C CNN "manf#"
+F 2 "Capacitor_SMD:CP_Elec_4x5.4" H 2150 1200 50  0001 C CNN
+F 3 "https://katalog.we-online.de/pbs/datasheet/865090440003.pdf" H 2150 1200 50  0001 C CNN
+F 4 "865090440003	" H 2150 1200 50  0001 C CNN "manf#"
 	1    2150 1200
 	1    0    0    -1
@@
 F 0 "C8" H 6891 1346 50  0000 L CNN
 F 1 "10uF" H 6891 1255 50  0000 L CNN
-F 2 "Capacitor_SMD:C_0805_2012Metric_Pad1.15x1.40mm_HandSolder" H 6800 1300 50  0001 C CNN
-F 3 "https://www.mouser.mx/datasheet/2/348/tct_p-951873.pdf" H 6800 1300 50  0001 C CNN
-F 4 "755-TCTP1C106M8R" H 6800 1300 50  0001 C CNN "manf#"
+F 2 "Capacitor_SMD:CP_Elec_4x5.4" H 6800 1300 50  0001 C CNN
+F 3 "https://katalog.we-online.de/pbs/datasheet/865090440003.pdf" H 6800 1300 50  0001 C CNN
+F 4 "865090440003	" H 6800 1300 50  0001 C CNN "manf#"
 	1    6800 1300
 	1    0    0    -1
@@
 F 0 "C5" H 3991 4646 50  0000 L CNN
 F 1 "10uF" H 3991 4555 50  0000 L CNN
-F 2 "Capacitor_SMD:C_0805_2012Metric_Pad1.15x1.40mm_HandSolder" H 3900 4600 50  0001 C CNN
-F 3 "https://www.mouser.mx/datasheet/2/348/tct_p-951873.pdf" H 3900 4600 50  0001 C CNN
-F 4 "755-TCTP1C106M8R" H 3900 4600 50  0001 C CNN "manf#"
+F 2 "Capacitor_SMD:C_Elec_4x5.4" H 3900 4600 50  0001 C CNN
+F 3 "https://katalog.we-online.de/pbs/datasheet/865090440003.pdf" H 3900 4600 50  0001 C CNN
+F 4 "865090440003	" H 3900 4600 50  0001 C CNN "manf#"
 	1    3900 4600
 	1    0    0    -1

Commit message: Last revision
Parts:
- removed R3, R4, R6: 1KOhm, Resistor_SMD:R_0805_2012Metric_Pad1.15x1.40mm_HandSolder, symbol Device:R_Small
Connections:
- net GND: no longer U1.1 (nSLEEP), U2.1 (nSLEEP), U3.1 (nSLEEP)
- net VCC: now also U1.1 (nSLEEP), U2.1 (nSLEEP), U3.1 (nSLEEP)
- no-connect marks 0 -> 4
Changed lines of the file:
@@
 Wire Wire Line
 	1650 1900 2050 1900
-$Comp
-L Driver_Motor:DRV8833PWP U1
-U 1 1 5D1CE3C8
-P 2650 2000
-F 0 "U1" H 2650 2881 50  0000 C CNN
-F 1 "DRV8833PWP" H 2650 2790 50  0000 C CNN
-F 2 "Package_SO:HTSSOP-16-1EP_4.4x5mm_P0.65mm_EP3.4x5mm_Mask2.46x2.31mm_ThermalVias" H 3100 2450 50  0001 L CNN
-F 3 "http://www.ti.com/lit/ds/symlink/drv8833.pdf" H 2500 2550 50  0001 C CNN
-F 4 "595-DRV8833CPWPR" H 2650 2000 50  0001 C CNN "manf#"
-	1    2650 2000
-	1    0    0    -1
-$EndComp
 Text Label 2050 2300 2    50   ~ 0
 GPIO4
@@
 Connection ~ 3600 4450
 $Comp
-L Motor:Motor_DC M3
-U 1 1 5D2161AE
-P 5800 4950
-F 0 "M3" H 5958 4946 50  0000 L CNN
-F 1 "Motor_DC" H 5958 4855 50  0000 L CNN
-F 2 "TerminalBlock:TerminalBlock_bornier-2_P5.08mm" H 5800 4860 50  0001 C CNN
-F 3 "~" H 5800 4860 50  0001 C CNN
-	1    5800 4950
-	1    0    0    -1
-$EndComp
-$Comp
 L Motor:Motor_DC M4
 U 1 1 5D2161B8
@@
 	1    0    0    -1
 $EndComp
-Text Label 5800 5250 0    50   ~ 0
-AFDER1
-Text Label 5800 4750 0    50   ~ 0
-AFDER2
 Text Label 5850 5500 0    50   ~ 0
 BFDER1
@@
 	4400 6300 4350 6300
 Connection ~ 4350 6300
-$Comp
-L Device:C_Small C6
-U 1 1 5D2161D5
-P 5100 4750
-F 0 "C6" H 5192 4796 50  0000 L CNN
-F 1 "2.2uF" H 5192 4705 50  0000 L CNN
-F 2 "Capacitor_SMD:C_0805_2012Metric_Pad1.15x1.40mm_HandSolder" H 5100 4750 50  0001 C CNN
-F 3 "https://www.mouser.mx/datasheet/2/445/885012107012-553996.pdf" H 5100 4750 50  0001 C CNN
-F 4 "710-885012107012" H 5100 4750 50  0001 C CNN "manf#"
-	1    5100 4750
-	1    0    0    -1
-$EndComp
 Wire Wire Line
 	4600 4700 4600 4650
 Wire Wire Line
 	4600 4650 5100 4650
-$Comp
-L power:GND #PWR011
-U 1 1 5D2161E1
-P 5100 4950
-F 0 "#PWR011" H 5100 4700 50  0001 C CNN
-F 1 "GND" H 5105 4777 50  0000 C CNN
-F 2 "" H 5100 4950 50  0001 C CNN
-F 3 "" H 5100 4950 50  0001 C CNN
-	1    5100 4950
-	1    0    0    -1
-$EndComp
 Wire Wire Line
 	5100 4850 5100 4950
@@
 GND
 $Comp
-L Device:R_Small R3
-U 1 1 5D23B9EF
-P 3550 1800
-F 0 "R3" H 3609 1846 50  0000 L CNN
-F 1 "1KOhm" H 3609 1755 50  0000 L CNN
-F 2 "Resistor_SMD:R_0805_2012Metric_Pad1.15x1.40mm_HandSolder" H 3550 1800 50  0001 C CNN
-F 3 "https://www.mouser.mx/datasheet/2/219/RN73H-12200.pdf" H 3550 1800 50  0001 C CNN
-F 4 "660-RN73H2ATD1001B25" H 3550 1800 50  0001 C CNN "manf#"
-	1    3550 1800
-	1    0    0    -1
-$EndComp
-Wire Wire Line
-	3250 1900 3550 1900
-Wire Wire Line
-	3550 1150 3550 1700
-$Comp
 L power:+12V #PWR02
 U 1 1 5D241FAE
@@
 	1    0    0    -1
 $EndComp
-$Comp
-L Device:R_Small R6
-U 1 1 5D24338F
-P 8200 1900
-F 0 "R6" H 8259 1946 50  0000 L CNN
-F 1 "1KOhm" H 8259 1855 50  0000 L CNN
-F 2 "Resistor_SMD:R_0805_2012Metric_Pad1.15x1.40mm_HandSolder" H 8200 1900 50  0001 C CNN
-F 3 "https://www.mouser.mx/datasheet/2/219/RN73H-12200.pdf" H 8200 1900 50  0001 C CNN
-F 4 "660-RN73H2ATD1001B25" H 8200 1900 50  0001 C CNN "manf#"
-	1    8200 1900
-	1    0    0    -1
-$EndComp
-Wire Wire Line
-	7900 2000 8200 2000
-Wire Wire Line
-	8200 1250 8200 1800
-$Comp
-L Device:R_Small R4
-U 1 1 5D247081
-P 5300 5200
-F 0 "R4" H 5359 5246 50  0000 L CNN
-F 1 "1KOhm" H 5359 5155 50  0000 L CNN
-F 2 "Resistor_SMD:R_0805_2012Metric_Pad1.15x1.40mm_HandSolder" H 5300 5200 50  0001 C CNN
-F 3 "https://www.mouser.mx/datasheet/2/219/RN73H-12200.pdf" H 5300 5200 50  0001 C CNN
-F 4 "660-RN73H2ATD1001B25" H 5300 5200 50  0001 C CNN "manf#"
-	1    5300 5200
-	1    0    0    -1
-$EndComp
-Wire Wire Line
-	5000 5300 5300 5300
-Wire Wire Line
-	5300 4550 5300 5100
-$Comp
-L power:GND #PWR0101
-U 1 1 5D24AE3D
-P 1600 1600
-F 0 "#PWR0101" H 1600 1350 50  0001 C CNN
-F 1 "GND" H 1605 1427 50  0000 C CNN
-F 2 "" H 1600 1600 50  0001 C CNN
-F 3 "" H 1600 1600 50  0001 C CNN
-	1    1600 1600
-	1    0    0    -1
-$EndComp
 Wire Wire Line
 	2050 1600 1600 1600
-$Comp
-L power:GND #PWR0102
-U 1 1 5D24D496
-P 6200 1700
-F 0 "#PWR0102" H 6200 1450 50  0001 C CNN
-F 1 "GND" H 6205 1527 50  0000 C CNN
-F 2 "" H 6200 1700 50  0001 C CNN
-F 3 "" H 6200 1700 50  0001 C CNN
-	1    6200 1700
-	1    0    0    -1
-$EndComp
 Wire Wire Line
 	6700 1700 6200 1700
-$Comp
-L power:GND #PWR0103
-U 1 1 5D251B75
-P 3200 5050
-F 0 "#PWR0103" H 3200 4800 50  0001 C CNN
-F 1 "GND" H 3205 4877 50  0000 C CNN
-F 2 "" H 3200 5050 50  0001 C CNN
-F 3 "" H 3200 5050 50  0001 C CNN
-	1    3200 5050
-	1    0    0    -1
-$EndComp
 Wire Wire Line
 	3800 5000 3200 5000
-Wire Wire Line
-	3200 5000 3200 5050
 $Comp
 L power:+12V #PWR0104
@@
 $EndComp
 $Comp
-L power:VCC #PWR0107
-U 1 1 5D27E53E
-P 8200 1250
-F 0 "#PWR0107" H 8200 1100 50  0001 C CNN
-F 1 "VCC" H 8217 1423 50  0000 C CNN
-F 2 "" H 8200 1250 50  0001 C CNN
-F 3 "" H 8200 1250 50  0001 C CNN
-	1    8200 1250
-	1    0    0    -1
-$EndComp
-$Comp
-L power:VCC #PWR0108
-U 1 1 5D27EC09
-P 3550 1150
-F 0 "#PWR0108" H 3550 1000 50  0001 C CNN
-F 1 "VCC" H 3567 1323 50  0000 C CNN
-F 2 "" H 3550 1150 50  0001 C CNN
-F 3 "" H 3550 1150 50  0001 C CNN
-	1    3550 1150
-	1    0    0    -1
-$EndComp
-$Comp
-L power:VCC #PWR0109
-U 1 1 5D27F5A5
-P 5300 4550
-F 0 "#PWR0109" H 5300 4400 50  0001 C CNN
-F 1 "VCC" H 5317 4723 50  0000 C CNN
-F 2 "" H 5300 4550 50  0001 C CNN
-F 3 "" H 5300 4550 50  0001 C CNN
-	1    5300 4550
-	1    0    0    -1
-$EndComp
-$Comp
 L Device:R_Small R7
 U 1 1 5D250BC0
@@
 Wire Wire Line
 	3200 5200 3800 5200
+$Comp
+L power:VCC #PWR0101
+U 1 1 5D3268F3
+P 1600 1600
+F 0 "#PWR0101" H 1600 1450 50  0001 C CNN
+F 1 "VCC" H 1617 1773 50  0000 C CNN
+F 2 "" H 1600 1600 50  0001 C CNN
+F 3 "" H 1600 1600 50  0001 C CNN
+	1    1600 1600
+	1    0    0    -1
+$EndComp
+$Comp
+L Driver_Motor:DRV8833PWP U1
+U 1 1 5D1CE3C8
+P 2650 2000
+F 0 "U1" H 2650 2881 50  0000 C CNN
+F 1 "DRV8833PWP" H 2650 2790 50  0000 C CNN
+F 2 "Package_SO:HTSSOP-16-1EP_4.4x5mm_P0.65mm_EP3.4x5mm_Mask2.46x2.31mm_ThermalVias" H 3100 2450 50  0001 L CNN
+F 3 "http://www.ti.com/lit/ds/symlink/drv8833.pdf" H 2500 2550 50  0001 C CNN
+F 4 "595-DRV8833CPWPR" H 2650 2000 50  0001 C CNN "manf#"
+	1    2650 2000
+	1    0    0    -1
+$EndComp
+$Comp
+L power:VCC #PWR0102
+U 1 1 5D3276DD
+P 6200 1700
+F 0 "#PWR0102" H 6200 1550 50  0001 C CNN
+F 1 "VCC" H 6217 1873 50  0000 C CNN
+F 2 "" H 6200 1700 50  0001 C CNN
+F 3 "" H 6200 1700 50  0001 C CNN
+	1    6200 1700
+	1    0    0    -1
+$EndComp
+NoConn ~ 7900 2000
+NoConn ~ 3250 1900
+$Comp
+L power:VCC #PWR0103
+U 1 1 5D32E8F4
+P 3200 5000
+F 0 "#PWR0103" H 3200 4850 50  0001 C CNN
+F 1 "VCC" H 3217 5173 50  0000 C CNN
+F 2 "" H 3200 5000 50  0001 C CNN
+F 3 "" H 3200 5000 50  0001 C CNN
+	1    3200 5000
+	1    0    0    -1
+$EndComp
+$Comp
+L power:GND #PWR011
+U 1 1 5D2161E1
+P 5100 4950
+F 0 "#PWR011" H 5100 4700 50  0001 C CNN
+F 1 "GND" H 5105 4777 50  0000 C CNN
+F 2 "" H 5100 4950 50  0001 C CNN
+F 3 "" H 5100 4950 50  0001 C CNN
+	1    5100 4950
+	1    0    0    -1
+$EndComp
+$Comp
+L Device:C_Small C6
+U 1 1 5D2161D5
+P 5100 4750
+F 0 "C6" H 5192 4796 50  0000 L CNN
+F 1 "2.2uF" H 5192 4705 50  0000 L CNN
+F 2 "Capacitor_SMD:C_0805_2012Metric_Pad1.15x1.40mm_HandSolder" H 5100 4750 50  0001 C CNN
+F 3 "https://www.mouser.mx/datasheet/2/445/885012107012-553996.pdf" H 5100 4750 50  0001 C CNN
+F 4 "710-885012107012" H 5100 4750 50  0001 C CNN "manf#"
+	1    5100 4750
+	1    0    0    -1
+$EndComp
+Text Label 5800 4750 0    50   ~ 0
+AFDER2
+Text Label 5800 5250 0    50   ~ 0
+AFDER1
+$Comp
+L Motor:Motor_DC M3
+U 1 1 5D2161AE
+P 5800 4950
+F 0 "M3" H 5958 4946 50  0000 L CNN
+F 1 "Motor_DC" H 5958 4855 50  0000 L CNN
+F 2 "TerminalBlock:TerminalBlock_bornier-2_P5.08mm" H 5800 4860 50  0001 C CNN
+F 3 "~" H 5800 4860 50  0001 C CNN
+	1    5800 4950
+	1    0    0    -1
+$EndComp
+NoConn ~ 5000 5300
+NoConn ~ 5250 3250
 $EndSCHEMATC

Commit message: Last revision pcb
Connections:
- net GPIO2 renamed GPIO12
Changed lines of the file:
@@
 GPIO4
 Text Label 2050 2200 2    50   ~ 0
-GPIO2
+GPIO12
 Wire Wire Line
 	1650 1900 2050 1900
@@
 GPIO4
 Text Label 2050 2400 2    50   ~ 0
-GPIO2
+GPIO12
 Text Label 8300 5100 0    50   ~ 0
 GPIO4
 Text Label 8300 5000 0    50   ~ 0
-GPIO2
+GPIO12
 $Comp
 L Device:C_Small C7
@@
 GPIO4
 Text Label 3800 5600 2    50   ~ 0
-GPIO2
+GPIO12
 Text Label 3800 5800 2    50   ~ 0
 GPIO15
