File: Hardware/rover_car/rover_car.sch (KiCad schematic (older format))
At the start: 26 parts, among them J1 Conn_01x06_Female, J3 Screw_Terminal_01x02, M1 Motor_DC, M2 Motor_DC, M3 Motor_DC, M4 Motor_DC, M5 Motor_DC, M6 Motor_DC, U1 DRV8833PWP, U2 DRV8833PWP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

Commit message: Update PCB version 1.0
Parts:
- R2, R4, R6: manf# (none) -> 667-ERJ-U6SFR20V
Changed lines of the file:
@@
 encoding utf-8
 Sheet 1 1
-Title "DRIVER DE ROVER"
-Date "2019-07-09"
+Title "Rover Motor Driver"
+Date "2019-08-02"
 Rev "0.1"
-Comp "ELECTRONIC CATS"
+Comp "Electronic Cats"
 Comment1 "EDGAR EMMANUEL CAPUCHINO ESCOBEDO"
-Comment2 ""
+Comment2 "Eduardo Contreras"
 Comment3 ""
 Comment4 ""
@@
 F 1 "200mOhms" V 1750 1850 50  0000 L CNN
 F 2 "Resistor_SMD:R_0805_2012Metric_Pad1.15x1.40mm_HandSolder" H 1650 2100 50  0001 C CNN
-F 3 "https://www.mouser.mx/datasheet/2/315/AOA0000C334-1314047.pdf" H 1650 2100 50  0001 C CNN
+F 3 "https://www.mouser.mx/datasheet/2/315/AOA0000C334-1314047.pdf<...>" H 1650 2100 50  0001 C CNN
 F 4 "667-ERJ-U6SFR20V" H 1650 2100 50  0001 C CNN "manf#"
 	1    1650 2100
@@
 F 1 "200mOhm" V 6380 1895 50  0000 L CNN
 F 2 "Resistor_SMD:R_0805_2012Metric_Pad1.15x1.40mm_HandSolder" H 6300 2200 50  0001 C CNN
-F 3 "https://www.mouser.mx/datasheet/2/315/AOA0000C334-1314047.pdf" H 6300 2200 50  0001 C CNN
+F 3 "https://www.mouser.mx/datasheet/2/315/AOA0000C334-1314047.pdf<...>" H 6300 2200 50  0001 C CNN
 F 4 "667-ERJ-U6SFR20V" H 6300 2200 50  0001 C CNN "manf#"
 	1    6300 2200
@@
 F 1 "200mOhm" V 3480 5190 50  0000 L CNN
 F 2 "Resistor_SMD:R_0805_2012Metric_Pad1.15x1.40mm_HandSolder" H 3400 5500 50  0001 C CNN
-F 3 "https://www.mouser.mx/datasheet/2/315/AOA0000C334-1314047.pdf" H 3400 5500 50  0001 C CNN
+F 3 "https://www.mouser.mx/datasheet/2/315/AOA0000C334-1314047.pdf<...>" H 3400 5500 50  0001 C CNN
 F 4 "667-ERJ-U6SFR20V" H 3400 5500 50  0001 C CNN "manf#"
 	1    3400 5500
@@
 F 1 "200mOhms" V 1250 1900 50  0000 L CNN
 F 2 "Resistor_SMD:R_0805_2012Metric_Pad1.15x1.40mm_HandSolder" H 1400 2100 50  0001 C CNN
-F 3 "~" H 1400 2100 50  0001 C CNN
+F 3 "https://www.mouser.mx/datasheet/2/315/AOA0000C334-1314047.pdf<...>" H 1400 2100 50  0001 C CNN
+F 4 "667-ERJ-U6SFR20V" H 0   0   50  0001 C CNN "manf#"
 	1    1400 2100
 	1    0    0    -1
@@
 F 1 "200mOhms" V 6075 1865 50  0000 L CNN
 F 2 "Resistor_SMD:R_0805_2012Metric_Pad1.15x1.40mm_HandSolder" H 6150 2200 50  0001 C CNN
-F 3 "~" H 6150 2200 50  0001 C CNN
+F 3 "https://www.mouser.mx/datasheet/2/315/AOA0000C334-1314047.pdf<...>" H 6150 2200 50  0001 C CNN
+F 4 "667-ERJ-U6SFR20V" H 0   0   50  0001 C CNN "manf#"
 	1    6150 2200
 	1    0    0    -1
@@
 F 1 "200mOhm" V 3110 5185 50  0000 L CNN
 F 2 "Resistor_SMD:R_0805_2012Metric_Pad1.15x1.40mm_HandSolder" H 3200 5500 50  0001 C CNN
-F 3 "~" H 3200 5500 50  0001 C CNN
+F 3 "https://www.mouser.mx/datasheet/2/315/AOA0000C334-1314047.pdf" H 3200 5500 50  0001 C CNN
+F 4 "667-ERJ-U6SFR20V" H 0   0   50  0001 C CNN "manf#"
 	1    3200 5500
 	1    0    0    -1

Commit message: save changes
Parts:
- C1, C4: manf# 710-885012207039 -> 885012207039
- J3, M1, M2, M3, M4, M5, M6: manf# (none) -> 39594-3002
- R3, R4, R5: value 200mOhm -> 200mOhms
Changed lines of the file:
@@
 F 2 "Capacitor_SMD:C_0805_2012Metric_Pad1.15x1.40mm_HandSolder" H 1850 1350 50  0001 C CNN
 F 3 "https://www.mouser.mx/datasheet/2/445/885012207039-554525.pdf" H 1850 1350 50  0001 C CNN
-F 4 "710-885012207039" H 1850 1350 50  0001 C CNN "manf#"
+F 4 "885012207039" H 1850 1350 50  0001 C CNN "manf#"
 	1    1850 1350
 	1    0    0    -1
@@
 F 2 "TerminalBlock:TerminalBlock_bornier-2_P5.08mm" H 4050 1460 50  0001 C CNN
 F 3 "~" H 4050 1460 50  0001 C CNN
+F 4 "39594-3002" H 0   0   50  0001 C CNN "manf#"
 	1    4050 1550
 	1    0    0    -1
@@
 F 2 "TerminalBlock:TerminalBlock_bornier-2_P5.08mm" H 4050 2210 50  0001 C CNN
 F 3 "~" H 4050 2210 50  0001 C CNN
+F 4 "39594-3002" H 0   0   50  0001 C CNN "manf#"
 	1    4050 2300
 	1    0    0    -1
@@
 F 2 "TerminalBlock:TerminalBlock_bornier-2_P5.08mm" H 8700 1560 50  0001 C CNN
 F 3 "~" H 8700 1560 50  0001 C CNN
+F 4 "39594-3002" H 0   0   50  0001 C CNN "manf#"
 	1    8700 1650
 	1    0    0    -1
@@
 F 2 "TerminalBlock:TerminalBlock_bornier-2_P5.08mm" H 8700 2310 50  0001 C CNN
 F 3 "~" H 8700 2310 50  0001 C CNN
+F 4 "39594-3002" H 0   0   50  0001 C CNN "manf#"
 	1    8700 2400
 	1    0    0    -1
@@
 P 6300 2200
 F 0 "R5" H 6315 2305 50  0000 L CNN
-F 1 "200mOhm" V 6380 1895 50  0000 L CNN
+F 1 "200mOhms" V 6380 1895 50  0000 L CNN
 F 2 "Resistor_SMD:R_0805_2012Metric_Pad1.15x1.40mm_HandSolder" H 6300 2200 50  0001 C CNN
 F 3 "https://www.mouser.mx/datasheet/2/315/AOA0000C334-1314047.pdf<...>" H 6300 2200 50  0001 C CNN
@@
 F 2 "Capacitor_SMD:C_0805_2012Metric_Pad1.15x1.40mm_HandSolder" H 3600 4750 50  0001 C CNN
 F 3 "https://www.mouser.mx/datasheet/2/445/885012207039-554525.pdf" H 3600 4750 50  0001 C CNN
-F 4 "710-885012207039" H 3600 4750 50  0001 C CNN "manf#"
+F 4 "885012207039" H 3600 4750 50  0001 C CNN "manf#"
 	1    3600 4750
 	1    0    0    -1
@@
 F 2 "TerminalBlock:TerminalBlock_bornier-2_P5.08mm" H 5800 5610 50  0001 C CNN
 F 3 "~" H 5800 5610 50  0001 C CNN
+F 4 "39594-3002" H 0   0   50  0001 C CNN "manf#"
 	1    5800 5700
 	1    0    0    -1
@@
 P 3400 5500
 F 0 "R3" H 3415 5600 50  0000 L CNN
-F 1 "200mOhm" V 3480 5190 50  0000 L CNN
+F 1 "200mOhms" V 3480 5190 50  0000 L CNN
 F 2 "Resistor_SMD:R_0805_2012Metric_Pad1.15x1.40mm_HandSolder" H 3400 5500 50  0001 C CNN
 F 3 "https://www.mouser.mx/datasheet/2/315/AOA0000C334-1314047.pdf<...>" H 3400 5500 50  0001 C CNN
@@
 F 2 "TerminalBlock:TerminalBlock_bornier-2_P5.08mm" H 1050 5750 50  0001 C CNN
 F 3 "~" H 1050 5750 50  0001 C CNN
+F 4 "39594-3002" H 0   0   50  0001 C CNN "manf#"
 	1    1050 5750
 	1    0    0    -1
@@
 P 3200 5500
 F 0 "R4" H 3210 5610 50  0000 L CNN
-F 1 "200mOhm" V 3110 5185 50  0000 L CNN
+F 1 "200mOhms" V 3110 5185 50  0000 L CNN
 F 2 "Resistor_SMD:R_0805_2012Metric_Pad1.15x1.40mm_HandSolder" H 3200 5500 50  0001 C CNN
 F 3 "https://www.mouser.mx/datasheet/2/315/AOA0000C334-1314047.pdf" H 3200 5500 50  0001 C CNN
@@
 F 2 "TerminalBlock:TerminalBlock_bornier-2_P5.08mm" H 5800 4860 50  0001 C CNN
 F 3 "~" H 5800 4860 50  0001 C CNN
+F 4 "39594-3002" H 0   0   50  0001 C CNN "manf#"
 	1    5800 4950
 	1    0    0    -1
