File: Hardware/cat_finder_main/cat_finder_main.kicad_pcb (KiCad board)
At the start: 2 copper layers, 85 x 70 mm, 35 parts, among them J1 BATT, J10 Analog, J2 BME280, J3 CSS811, J4 DRIVERS, J5 GY-87, J6 PROG, J7 FTDI, J8 Digital, J9 i2c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

Commit message: add pin bast
Parts:
- added J11: Bast Pin, Connector_PinSocket_2.54mm:PinSocket_1x05_P2.54mm_Vertical, F.Cu at (110.7, 66.9)
- moved J4 4.27 mm to (124.1, 66.9)
- moved G*** 4.24 mm to (110.0, 71.7)
- moved JP1 1.64 mm to (124.2, 72.8)
- moved JP3 1.61 mm to (126.7, 72.8)
- moved JP4 1.56 mm to (129.2, 72.8)
- moved JP2 1.52 mm to (131.7, 72.8)
- moved D1 1.20 mm to (168.1, 96.2)
- moved JP10 0.11 mm to (143.5, 72.8)
Connections:
- JP7 pad 1: /A1 -> /A2
- JP8 pad 1: /11 -> /A1
Routing:
- net /10: track 0.00 -> 85.1 mm, vias 0 -> 2
- net /12: track 0.00 -> 82.1 mm, vias 0 -> 2
- net /13: track 0.00 -> 80.8 mm, vias 0 -> 2
- net /A0: track 0.00 -> 78.4 mm, vias 0 -> 2
- net /A2: track 0.00 -> 70.1 mm
- net /11: track 55.4 -> 83.4 mm, vias 0 -> 2
- net /A1: track 61.4 -> 73.7 mm
- net /A3: track 61.6 -> 68.6 mm
- net /GPIO14: track 41.1 -> 35.9 mm
- net /GPIO15: track 33.9 -> 29.8 mm
- net VCC: track 141.2 -> 143.0 mm
- net /GPIO12: track 18.9 -> 20.7 mm
- net /BATT: track 23.2 -> 24.9 mm
- net +3V3: track 188.1 -> 189.6 mm
- net /GPIO13: track 26.6 -> 25.2 mm
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