File: Hardware/cat_finder_main/cat_finder_main.kicad_pcb (KiCad board)
At the start: 2 copper layers, 85 x 70 mm, 37 parts, among them J1 BATT, J10 Analog, J11 Bast Pin, J2 BME280, J3 CSS811, J4 DRIVERS, J5 GY-87, J6 PROG, J7 FTDI, J8 Digital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

Commit message: delete d1
Parts:
- removed D1: 1N5817, Diode_THT:D_DO-41_SOD81_P10.16mm_Horizontal
- moved Q1 7.34 mm to (171.0, 81.1), turned to 90 degrees
- moved C3 6.70 mm to (167.9, 86.6), turned to 0 degrees
- moved R2 0.91 mm to (167.1, 69.6)
Connections:
- U2 pad 1: Net-(D1-Pad1) -> VCC
Routing:
- net VCC: track 74.3 -> 65.6 mm
- net Net-(D1-Pad1): track 8.13 -> 0.00 mm
- net /BATT: track 30.3 -> 24.8 mm

Commit message: change transistor pcb
Parts:
- Q1: value Q_PMOS_GDS -> Q_PMOS_DGS; footprint Package_TO_SOT_THT:TO-220-3_Vertical -> Package_TO_SOT_THT:TO-92_Inline
- moved Q1 5.10 mm to (171.0, 76.0), turned to 270 degrees
Routing:
- net VCC: track 65.6 -> 64.2 mm
Changed lines of the file:
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@@
     (thickness 1.6)
     (drawings 126)
-    (tracks 332)
+    (tracks 331)
     (zones 0)
     (modules 36)
@@
   (page A4)
   (layers
-    (0 F.Cu signal hide)
-    (31 B.Cu signal hide)
+    (0 F.Cu signal)
+    (31 B.Cu signal)
     (32 B.Adhes user)
     (33 F.Adhes user)
@@
     (add_net VCC)
   )
+  (module Package_TO_SOT_THT:TO-92_Inline (layer F.Cu)
+    (at 171 76 270)
+    (descr "TO-92 leads in-line, narrow, oval pads, drill 0.75mm (see NXP sot054_po.pdf)")
+    (tags "to-92 sc-43 sc-43a sot54 PA33 transistor")
+    (fp_text reference Q1 (at 1.27 -3.56 270) (layer F.SilkS)
+      (effects (font (size 1 1) (thickness 0.15)))
+    )
+    (fp_text value Q_PMOS_DGS (at 1.27 2.79 270) (layer F.Fab)
+      (effects (font (size 1 1) (thickness 0.15)))
+    )
+    (fp_arc (start 1.27 0) (end 1.27 -2.6) (angle 135) (layer F.SilkS) (width 0.12))
+    (fp_arc (start 1.27 0) (end 1.27 -2.48) (angle -135) (layer F.Fab) (width 0.1))
+    (fp_arc (start 1.27 0) (end 1.27 -2.6) (angle -135) (layer F.SilkS) (width 0.12))
+    (fp_arc (start 1.27 0) (end 1.27 -2.48) (angle 135) (layer F.Fab) (width 0.1))
+    (fp_line (start 4 2.01) (end -1.46 2.01) (layer F.CrtYd) (width 0.05))
+    (fp_line (start 4 2.01) (end 4 -2.73) (layer F.CrtYd) (width 0.05))
+    (fp_line (start -1.46 -2.73) (end -1.46 2.01) (layer F.CrtYd) (width 0.05))
+    (fp_line (start -1.46 -2.73) (end 4 -2.73) (layer F.CrtYd) (width 0.05))
+    (fp_line (start -0.5 1.75) (end 3 1.75) (layer F.Fab) (width 0.1))
+    (fp_line (start -0.53 1.85) (end 3.07 1.85) (layer F.SilkS) (width 0.12))
+    (fp_text user %R (at 1.27 -3.56 270) (layer F.Fab)
+      (effects (font (size 1 1) (thickness 0.15)))
+    )
+    (pad 3 thru_hole rect (at 0 0 270) (size 1.05 1.5) (drill 0.75) (layers *.Cu *.Mask)
+      (net 5 /BATT))
+    (pad 1 thru_hole oval (at 2.54 0 270) (size 1.05 1.5) (drill 0.75) (layers *.Cu *.Mask)
+      (net 3 VCC))
+    (pad 2 thru_hole oval (at 1.27 0 270) (size 1.05 1.5) (drill 0.75) (layers *.Cu *.Mask)
+      (net 3 VCC))
+    (model ${KISYS3DMOD}/Package_TO_SOT_THT.3dshapes/TO-92_Inline.wrl
+      (at (xyz 0 0 0))
+      (scale (xyz 1 1 1))
+      (rotate (xyz 0 0 0))
+    )
+  )
   (module Resistor_THT:R_Axial_DIN0207_L6.3mm_D2.5mm_P10.16mm_Horizontal (layer F.Cu)
     (at 167.1 69.6)
@@
     )
   )
-  (module Package_TO_SOT_THT:TO-220-3_Vertical (layer F.Cu)
-    (at 171 81.1 90)
-    (descr "TO-220-3, Vertical, RM 2.54mm, see https://www.vishay.com/docs/66542/to-220-1.pdf")
-    (tags "TO-220-3 Vertical RM 2.54mm")
-    (fp_text reference Q1 (at 9 -2.1 180) (layer F.SilkS)
-      (effects (font (size 1 1) (thickness 0.15)))
-    )
-    (fp_text value Q_PMOS_GDS (at 2.54 2.5 90) (layer F.Fab)
-      (effects (font (size 1 1) (thickness 0.15)))
-    )
-    (fp_text user %R (at 2.54 -4.27 90) (layer F.Fab)
-      (effects (font (size 1 1) (thickness 0.15)))
-    )
-    (fp_line (start 7.79 -3.4) (end -2.71 -3.4) (layer F.CrtYd) (width 0.05))
-    (fp_line (start 7.79 1.51) (end 7.79 -3.4) (layer F.CrtYd) (width 0.05))
-    (fp_line (start -2.71 1.51) (end 7.79 1.51) (layer F.CrtYd) (width 0.05))
-    (fp_line (start -2.71 -3.4) (end -2.71 1.51) (layer F.CrtYd) (width 0.05))
-    (fp_line (start 4.391 -3.27) (end 4.391 -1.76) (layer F.SilkS) (width 0.12))
-    (fp_line (start 0.69 -3.27) (end 0.69 -1.76) (layer F.SilkS) (width 0.12))
-    (fp_line (start -2.58 -1.76) (end 7.66 -1.76) (layer F.SilkS) (width 0.12))
-    (fp_line (start 7.66 -3.27) (end 7.66 1.371) (layer F.SilkS) (width 0.12))
-    (fp_line (start -2.58 -3.27) (end -2.58 1.371) (layer F.SilkS) (width 0.12))
-    (fp_line (start -2.58 1.371) (end 7.66 1.371) (layer F.SilkS) (width 0.12))
-    (fp_line (start -2.58 -3.27) (end 7.66 -3.27) (layer F.SilkS) (width 0.12))
-    (fp_line (start 4.39 -3.15) (end 4.39 -1.88) (layer F.Fab) (width 0.1))
-    (fp_line (start 0.69 -3.15) (end 0.69 -1.88) (layer F.Fab) (width 0.1))
-    (fp_line (start -2.46 -1.88) (end 7.54 -1.88) (layer F.Fab) (width 0.1))
-    (fp_line (start 7.54 -3.15) (end -2.46 -3.15) (layer F.Fab) (width 0.1))
-    (fp_line (start 7.54 1.25) (end 7.54 -3.15) (layer F.Fab) (width 0.1))
-    (fp_line (start -2.46 1.25) (end 7.54 1.25) (layer F.Fab) (width 0.1))
-    (fp_line (start -2.46 -3.15) (end -2.46 1.25) (layer F.Fab) (width 0.1))
-    (pad 3 thru_hole oval (at 5.08 0 90) (size 1.905 2) (drill 1.1) (layers *.Cu *.Mask)
-      (net 5 /BATT))
-    (pad 2 thru_hole oval (at 2.54 0 90) (size 1.905 2) (drill 1.1) (layers *.Cu *.Mask)
-      (net 3 VCC))
-    (pad 1 thru_hole rect (at 0 0 90) (size 1.905 2) (drill 1.1) (layers *.Cu *.Mask)
-      (net 3 VCC))
-    (model ${KISYS3DMOD}/Package_TO_SOT_THT.3dshapes/TO-220-3_Vertical.wrl
-      (at (xyz 0 0 0))
-      (scale (xyz 1 1 1))
-      (rotate (xyz 0 0 0))
-    )
-  )
   (module Connector_PinSocket_2.54mm:PinSocket_1x05_P2.54mm_Vertical (layer F.Cu)
     (at 110.7 66.9 90)
@@
   (segment (start 169.2 104.3) (end 170.8 104.3) (width 0.5) (layer F.Cu) (net 3))
   (segment (start 168.6 104.9) (end 169.2 104.3) (width 0.5) (layer F.Cu) (net 3))
-  (segment (start 168 81.1) (end 171 81.1) (width 0.5) (layer B.Cu) (net 3))
-  (segment (start 171 78.56) (end 171 81.1) (width 0.5) (layer B.Cu) (net 3))
-  (segment (start 171 85.2) (end 171 81.1) (width 0.5) (layer B.Cu) (net 3))
-  (segment (start 169.6 86.6) (end 171 85.2) (width 0.5) (layer B.Cu) (net 3))
-  (segment (start 167.9 86.6) (end 169.6 86.6) (width 0.5) (layer B.Cu) (net 3))
   (segment (start 167.9 92.05) (end 168.05 92.2) (width 0.5) (layer B.Cu) (net 3))
   (segment (start 167.9 86.6) (end 167.9 92.05) (width 0.5) (layer B.Cu) (net 3))
@@
   (segment (start 162.53 64.4) (end 166.1 64.4) (width 0.5) (layer B.Cu) (net 3))
   (segment (start 166.1 64.4) (end 167.1 65.4) (width 0.5) (layer B.Cu) (net 3))
-  (segment (start 167.1 80.2) (end 167.6 80.7) (width 0.5) (layer B.Cu) (net 3))
-  (segment (start 167.1 69.6) (end 167.1 80.2) (width 0.5) (layer B.Cu) (net 3))
-  (segment (start 167.6 80.7) (end 168 81.1) (width 0.5) (layer B.Cu) (net 3))
+  (segment (start 171 77.27) (end 171 78.54) (width 0.5) (layer B.Cu) (net 3))
+  (segment (start 169.6 86.6) (end 167.9 86.6) (width 0.5) (layer B.Cu) (net 3))
+  (segment (start 171 78.54) (end 171 85.2) (width 0.5) (layer B.Cu) (net 3))
+  (segment (start 171 85.2) (end 169.6 86.6) (width 0.5) (layer B.Cu) (net 3))
+  (segment (start 168.24 78.54) (end 171 78.54) (width 0.5) (layer B.Cu) (net 3))
+  (segment (start 167.1 77.4) (end 168.24 78.54) (width 0.5) (layer B.Cu) (net 3))
+  (segment (start 167.1 69.6) (end 167.1 77.4) (width 0.5) (layer B.Cu) (net 3))
   (segment (start 112.34 120.46) (end 112.3 120.5) (width 0.3) (layer B.Cu) (net 4))
   (segment (start 112.34 114.4) (end 112.34 120.46) (width 0.3) (layer B.Cu) (net 4))
@@
   (segment (start 171.0475 76.02) (end 171.0675 76) (width 0.5) (layer B.Cu) (net 5))
   (segment (start 171 76.02) (end 171.0475 76.02) (width 0.5) (layer B.Cu) (net 5))
-  (segment (start 171.0675 76) (end 173.1 76) (width 0.5) (layer B.Cu) (net 5))
   (segment (start 173.1 76) (end 174.1 77) (width 0.5) (layer B.Cu) (net 5))
   (segment (start 174.1 77) (end 174.1 83.3) (width 0.5) (layer B.Cu) (net 5))
   (segment (start 175.58 84.78) (end 179.4 84.78) (width 0.5) (layer B.Cu) (net 5))
   (segment (start 174.1 83.3) (end 175.58 84.78) (width 0.5) (layer B.Cu) (net 5))
+  (segment (start 173.1 76) (end 171 76) (width 0.5) (layer B.Cu) (net 5))
   (segment (start 154.89 114.41) (end 154.98 114.5) (width 0.3) (layer F.Cu) (net 6))
   (segment (start 154.89 108.92) (end 154.89 114.41) (width 0.3) (layer F.Cu) (net 6))

Commit message: Update diode
Parts:
- added D1: SB260-E3/54, Diode_THT:D_A-405_P7.62mm_Horizontal, F.Cu at (174.2, 83.1)
- moved Q1 2.80 mm to (171.0, 73.2)
Connections:
- C1 pad 1: VCC -> Net-(C1-Pad1)
- J10 pad 9: Net-(J10-Pad9) -> +3V3
- Q1 pad 1: VCC -> Net-(C1-Pad1)
- U1 pad 3: VCC -> Net-(C1-Pad1)
Routing:
- net +3V3: track 147.9 -> 200.1 mm
- net Net-(C1-Pad1): track 0.00 -> 46.6 mm
- net VCC: track 64.2 -> 38.9 mm
- net /BATT: track 24.9 -> 28.4 mm
