File: Hardware/cat_finder_main/cat_finder_main.sch (KiCad schematic (older format))
At the start: 31 parts, among them J1 BATT, J10 Analog, J11 Bast Pin, J2 BME280, J3 CSS811, J4 DRIVERS, J5 GY-87, J6 PROG, J7 FTDI, J8 Digital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

Commit message: change diode´s name
Parts:
- D1, D3: value D_Schottky -> SB260
- D4: value D_Schottky -> 1N5817
Changed lines of the file:
@@
 EESchema Schematic File Version 4
-LIBS:cat_finder_main-cache
 EELAYER 29 0
 EELAYER END
@@
 P 1700 1330
 F 0 "D1" V 1746 1251 50  0000 R CNN
-F 1 "D_Schottky" V 1655 1251 50  0000 R CNN
+F 1 "SB260" V 1655 1251 50  0000 R CNN
 F 2 "Diode_THT:D_A-405_P10.16mm_Horizontal" H 1700 1330 50  0001 C CNN
 F 3 "https://www.mouser.mx/datasheet/2/427/sb220-104141.pdf" H 1700 1330 50  0001 C CNN
@@
 P 9330 4510
 F 0 "D3" V 9376 4431 50  0000 R CNN
-F 1 "D_Schottky" V 9285 4431 50  0000 R CNN
+F 1 "SB260" V 9285 4431 50  0000 R CNN
 F 2 "Diode_THT:D_A-405_P10.16mm_Horizontal" H 9330 4510 50  0001 C CNN
 F 3 "https://www.mouser.mx/datasheet/2/427/sb220-104141.pdf" H 9330 4510 50  0001 C CNN
@@
 P 1400 1330
 F 0 "D4" V 1450 1670 50  0000 R CNN
-F 1 "D_Schottky" V 1350 1830 50  0000 R CNN
+F 1 "1N5817" V 1360 1750 50  0000 R CNN
 F 2 "Diode_THT:D_DO-41_SOD81_P10.16mm_Horizontal" H 1400 1330 50  0001 C CNN
 F 3 "mouser.mx/datasheet/2/345/1n5817-1n5819-24580.pdf" H 1400 1330 50  0001 C CNN

Commit message: Add MOSFET
Parts:
- removed D1, D3: SB260, Diode_THT:D_A-405_P10.16mm_Horizontal, symbol Device:D_Schottky
- added Q1: Q_PMOS_GDS, Package_TO_SOT_THT:TO-220-3_Vertical, symbol Device:Q_PMOS_GDS
- added R2: 47k, Resistor_THT:R_Axial_DIN0207_L6.3mm_D2.5mm_P10.16mm_Horizontal, symbol Device:R
- renumbered D4 to D1
Connections:
- wire segments 79 -> 81
- no-connect marks 6 -> 7
Other:
- moved on the sheet: C1, C2, C3, D1, SW1A, U1, U2

Commit message: delete d1
Parts:
- removed D1: 1N5817, Diode_THT:D_DO-41_SOD81_P10.16mm_Horizontal, symbol Device:D_Schottky
Connections:
- wire segments 81 -> 80
Changed lines of the file:
@@
 	1    0    0    -1
 $EndComp
-Wire Wire Line
-	3630 3680 3830 3680
 $Comp
 L power:GND #PWR06
@@
 NoConn ~ 8980 4790
 $Comp
-L Device:D_Schottky D1
-U 1 1 5D782221
-P 3980 3680
-F 0 "D1" H 4030 3580 50  0000 R CNN
-F 1 "1N5817" H 4130 3790 50  0000 R CNN
-F 2 "Diode_THT:D_DO-41_SOD81_P10.16mm_Horizontal" H 3980 3680 50  0001 C CNN
-F 3 "mouser.mx/datasheet/2/345/1n5817-1n5819-24580.pdf" H 3980 3680 50  0001 C CNN
-F 4 "1N5817-T" V 3980 3680 50  0001 C CNN "manf#"
-	1    3980 3680
-	-1   0    0    1
-$EndComp
-$Comp
 L Device:Q_PMOS_GDS Q1
 U 1 1 5D7B7439
@@
 	1380 1690 2380 1690
 Wire Wire Line
-	4130 3680 4220 3680
-Wire Wire Line
 	3630 3880 4220 3880
 $Comp
@@
 Wire Wire Line
 	1380 2110 1380 2220
+Wire Wire Line
+	3630 3680 4220 3680
 $EndSCHEMATC

Commit message: change transistor
Parts:
- removed Q1: Q_PMOS_GDS, Package_TO_SOT_THT:TO-220-3_Vertical, symbol Device:Q_PMOS_GDS
- added Q?: Q_PMOS_DGS, Package_TO_SOT_THT:TO-92_Inline, symbol Device:Q_PMOS_DGS
Changed lines of the file:
@@
 NoConn ~ 8980 4790
-$Comp
-L Device:Q_PMOS_GDS Q1
-U 1 1 5D7B7439
-P 2280 1210
-F 0 "Q1" H 2486 1164 50  0000 L CNN
-F 1 "Q_PMOS_GDS" H 2486 1255 50  0000 L CNN
-F 2 "Package_TO_SOT_THT:TO-220-3_Vertical" H 2480 1310 50  0001 C CNN
-F 3 "https://www.mouser.mx/datasheet/2/308/NDP6020P-1306840.pdf" H 2280 1210 50  0001 C CNN
-F 4 "NDP6020P" H 2280 1210 50  0001 C CNN "manf#"
-	1    2280 1210
-	1    0    0    1
-$EndComp
 $Comp
 L power:VCC #PWR04
@@
 Wire Wire Line
 	3630 3680 4220 3680
+$Comp
+L Device:Q_PMOS_DGS Q?
+U 1 1 5D7BFB03
+P 2280 1210
+F 0 "Q?" H 2486 1164 50  0000 L CNN
+F 1 "Q_PMOS_DGS" H 2486 1255 50  0000 L CNN
+F 2 "Package_TO_SOT_THT:TO-92_Inline" H 2480 1310 50  0001 C CNN
+F 3 "https://www.mouser.mx/datasheet/2/268/TP2104%20C081313-846395.pdf" H 2280 1210 50  0001 C CNN
+F 4 "TP2104N3-G" H 2280 1210 50  0001 C CNN "manf#"
+	1    2280 1210
+	1    0    0    1
+$EndComp
 $EndSCHEMATC

Commit message: change transistor pcb
Parts:
- gave numbers to parts that had none: 1
Changed lines of the file:
@@
 	3630 3680 4220 3680
 $Comp
-L Device:Q_PMOS_DGS Q?
+L Device:Q_PMOS_DGS Q1
 U 1 1 5D7BFB03
 P 2280 1210
-F 0 "Q?" H 2486 1164 50  0000 L CNN
+F 0 "Q1" H 2486 1164 50  0000 L CNN
 F 1 "Q_PMOS_DGS" H 2486 1255 50  0000 L CNN
 F 2 "Package_TO_SOT_THT:TO-92_Inline" H 2480 1310 50  0001 C CNN

Commit message: Update diode
Parts:
- added D1: SB260-E3/54, Diode_THT:D_A-405_P7.62mm_Horizontal, symbol Device:D_Schottky
Connections:
- net +3V3: now also J10.9 (Pin_9)
- net VCC: now also D1.2 (A); no longer C1.1, Q1.1 (D), U1.3 (VI)
- new net: C1.1, D1.1 (K), Q1.1 (D), U1.3 (VI)
- no-connect marks 7 -> 6
Changed lines of the file:
@@
 	2380 2190 3280 2190
-Wire Wire Line
-	2980 1690 2380 1690
-Connection ~ 2380 1690
-Wire Wire Line
-	2380 1690 2380 1790
 Wire Wire Line
 	3980 1990 3980 2190
@@
 Text Label 10300 5900 2    50   ~ 0
 A0
-NoConn ~ 8980 4790
 $Comp
 L power:VCC #PWR04
@@
 Wire Wire Line
 	2380 1010 2380 910
-Wire Wire Line
-	2380 1410 2380 1690
-Wire Wire Line
-	1380 1690 1380 1210
 Connection ~ 1380 1210
 Wire Wire Line
@@
 Wire Wire Line
 	1380 1210 2080 1210
-Wire Wire Line
-	1380 1690 2380 1690
 Wire Wire Line
 	3630 3880 4220 3880
@@
 	1    0    0    -1
 $EndComp
-Wire Wire Line
-	1380 1810 1380 1690
-Connection ~ 1380 1690
 Wire Wire Line
 	1380 2110 1380 2220
@@
 	1    0    0    1
 $EndComp
+$Comp
+L Device:D_Schottky D1
+U 1 1 5D7ED820
+P 1890 1690
+F 0 "D1" H 1890 1474 50  0000 C CNN
+F 1 "SB260-E3/54" H 1890 1565 50  0000 C CNN
+F 2 "Diode_THT:D_A-405_P7.62mm_Horizontal" H 1890 1690 50  0001 C CNN
+F 3 "~" H 1890 1690 50  0001 C CNN
+F 4 "SB260-E3/54" H 1890 1690 50  0001 C CNN "manf#"
+	1    1890 1690
+	-1   0    0    1
+$EndComp
+Wire Wire Line
+	1380 1210 1380 1690
+Wire Wire Line
+	1740 1690 1380 1690
+Connection ~ 1380 1690
+Wire Wire Line
+	1380 1690 1380 1810
+Wire Wire Line
+	2380 1410 2380 1690
+Wire Wire Line
+	2040 1690 2380 1690
+Connection ~ 2380 1690
+Wire Wire Line
+	2380 1690 2380 1790
+Wire Wire Line
+	2380 1690 2980 1690
+$Comp
+L power:+3.3V #PWR?
+U 1 1 5D8098BD
+P 9305 4665
+F 0 "#PWR?" H 9305 4515 50  0001 C CNN
+F 1 "+3.3V" H 9320 4838 50  0000 C CNN
+F 2 "" H 9305 4665 50  0001 C CNN
+F 3 "" H 9305 4665 50  0001 C CNN
+	1    9305 4665
+	1    0    0    -1
+$EndComp
+Wire Wire Line
+	8980 4790 9305 4790
+Wire Wire Line
+	9305 4790 9305 4665
 $EndSCHEMATC
